File: pcb/reflow_controller_v2.sch (EAGLE design)
At the start: 88 parts, among them Q1 IRLML2502, Q2 IRLML2502, Q4 IRLML2502, Q5 IRLML2502, Q6 IRLML2502, U1 MAX6675, U10 MLT-5030-BUZZER, U11 HILINK_PM03, U2 MAX6675, U3 RT9193_SC70-5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

Commit message: updated schematics and code
Other:
- note added: "ESP32 S2"
- note removed: "ESP32 PICO D4"
Changed lines of the file:
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@@
 <setting verticaltext="up"/>
 </settings>
-<grid distance="0.1" unitdist="inch" unit="inch" style="lines" multiple="1" display="no" altdistance="0.01" altunitdist="inch" altunit="inch"/>
+<grid distance="0.1" unitdist="inch" unit="inch" style="lines" multiple="1" display="yes" altdistance="0.01" altunitdist="inch" altunit="inch"/>
 <layers>
 <layer number="1" name="Top" color="4" fill="1" visible="no" active="no"/>
@@
 <wire x1="99.06" y1="71.12" x2="99.06" y2="5.08" width="0.1524" layer="97"/>
 <wire x1="152.4" y1="71.12" x2="152.4" y2="5.08" width="0.1524" layer="97"/>
-<text x="314.96" y="251.46" size="2.54" layer="94" font="vector" align="center">ESP32 PICO D4</text>
+<text x="314.96" y="251.46" size="2.54" layer="94" font="vector" align="center">ESP32 S2</text>
 <wire x1="231.14" y1="71.12" x2="231.14" y2="5.08" width="0.1524" layer="97"/>
 <wire x1="289.56" y1="71.12" x2="289.56" y2="25.4" width="0.1524" layer="97"/>
